File: LED-driver-kicad/Ethernet.kicad_sch (KiCad schematic)
At the start: 23 parts, among them J1 ARJM11C7-114-BA-EW2, U1 ENC28J60x-SO, Y1 25MHz

Commit message: update footprint assignments
Parts:
- C1, C13, C14, C15, C2, C3, C4, C6: footprint (none) -> Capacitor_SMD:C_0402_1005Metric
- R13, R14, R15, R4, R6: footprint (none) -> Resistor_SMD:R_0402_1005Metric
Changed lines of the file:
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@@
       (effects (font (size 1.27 1.27)) (justify left))
     )
-    (property "Footprint" "" (at 222.25 79.375 0)
+    (property "Footprint" "Resistor_SMD:R_0402_1005Metric" (at 222.25 79.375 0)
       (effects (font (size 1.27 1.27)) hide)
     )
@@
       (effects (font (size 1.27 1.27)) (justify left))
     )
-    (property "Footprint" "" (at 243.205 88.265 0)
+    (property "Footprint" "Capacitor_SMD:C_0402_1005Metric" (at 243.205 88.265 0)
       (effects (font (size 1.27 1.27)) hide)
     )
@@
       (effects (font (size 1.27 1.27)) (justify left))
     )
-    (property "Footprint" "" (at 143.51 36.195 0)
+    (property "Footprint" "Capacitor_SMD:C_0402_1005Metric" (at 143.51 36.195 0)
       (effects (font (size 1.27 1.27)) hide)
     )
@@
       (effects (font (size 1.27 1.27)) (justify left))
     )
-    (property "Footprint" "" (at 115.57 68.58 0)
+    (property "Footprint" "Capacitor_SMD:C_0402_1005Metric" (at 115.57 68.58 0)
       (effects (font (size 1.27 1.27)) hide)
     )
@@
       (effects (font (size 1.27 1.27)) (justify right))
     )
-    (property "Footprint" "" (at 208.915 96.52 0)
+    (property "Footprint" "Resistor_SMD:R_0402_1005Metric" (at 208.915 96.52 0)
       (effects (font (size 1.27 1.27)) hide)
     )
@@
       (effects (font (size 1.27 1.27)) (justify left))
     )
-    (property "Footprint" "" (at 111.125 36.195 0)
+    (property "Footprint" "Capacitor_SMD:C_0402_1005Metric" (at 111.125 36.195 0)
       (effects (font (size 1.27 1.27)) hide)
     )
@@
       (effects (font (size 1.27 1.27)) (justify left))
     )
-    (property "Footprint" "" (at 222.25 86.995 0)
+    (property "Footprint" "Resistor_SMD:R_0402_1005Metric" (at 222.25 86.995 0)
       (effects (font (size 1.27 1.27)) hide)
     )
@@
       (effects (font (size 1.27 1.27)))
     )
-    (property "Footprint" "" (at 120.65 84.455 0)
+    (property "Footprint" "Capacitor_SMD:C_0402_1005Metric" (at 120.65 84.455 0)
       (effects (font (size 1.27 1.27)) hide)
     )
@@
       (effects (font (size 1.27 1.27)))
     )
-    (property "Footprint" "" (at 216.535 59.055 0)
+    (property "Footprint" "Resistor_SMD:R_0402_1005Metric" (at 216.535 59.055 0)
       (effects (font (size 1.27 1.27)) hide)
     )
@@
       (effects (font (size 1.27 1.27)))
     )
-    (property "Footprint" "" (at 205.105 41.275 0)
+    (property "Footprint" "Resistor_SMD:R_0402_1005Metric" (at 205.105 41.275 0)
       (effects (font (size 1.27 1.27)) hide)
     )
@@
       (effects (font (size 1.27 1.27)))
     )
-    (property "Footprint" "" (at 158.75 47.625 0)
+    (property "Footprint" "Resistor_SMD:R_0402_1005Metric" (at 158.75 47.625 0)
       (effects (font (size 1.27 1.27)) hide)
     )
@@
       (effects (font (size 1.27 1.27)))
     )
-    (property "Footprint" "" (at 205.105 32.385 0)
+    (property "Footprint" "Resistor_SMD:R_0402_1005Metric" (at 205.105 32.385 0)
       (effects (font (size 1.27 1.27)) hide)
     )
@@
       (effects (font (size 1.27 1.27)))
     )
-    (property "Footprint" "" (at 120.65 74.295 0)
+    (property "Footprint" "Capacitor_SMD:C_0402_1005Metric" (at 120.65 74.295 0)
       (effects (font (size 1.27 1.27)) hide)
     )
@@
       (effects (font (size 1.27 1.27)) (justify left))
     )
-    (property "Footprint" "" (at 200.025 96.52 0)
+    (property "Footprint" "Capacitor_SMD:C_0402_1005Metric" (at 200.025 96.52 0)
       (effects (font (size 1.27 1.27)) hide)
     )
@@
       (effects (font (size 1.27 1.27)) (justify left))
     )
-    (property "Footprint" "" (at 133.35 36.195 0)
+    (property "Footprint" "Capacitor_SMD:C_0402_1005Metric" (at 133.35 36.195 0)
       (effects (font (size 1.27 1.27)) hide)
     )
@@
       (effects (font (size 1.27 1.27)) (justify left))
     )
-    (property "Footprint" "" (at 236.855 59.055 0)
+    (property "Footprint" "Capacitor_SMD:C_0402_1005Metric" (at 236.855 59.055 0)
       (effects (font (size 1.27 1.27)) hide)
     )
@@
       (effects (font (size 1.27 1.27)) (justify left))
     )
-    (property "Footprint" "" (at 121.285 36.195 0)
+    (property "Footprint" "Capacitor_SMD:C_0402_1005Metric" (at 121.285 36.195 0)
       (effects (font (size 1.27 1.27)) hide)
     )
@@
       (effects (font (size 1.27 1.27)) (justify left))
     )
-    (property "Footprint" "" (at 216.535 51.435 0)
-      (effects (font (size 1.27 1.27)) hide)
-    )
+    (property "Footprint" "Resistor_SMD:R_0402_1005Metric" (at 216.535 51.435 0)
+      (effects (font (size 1.27 1.27)) hide)
+    )

Commit message: update footprint assignments
Parts:
- removed R16: R_Small, symbol Device:R_Small
- J1: footprint Connector_RJ:Connector_RJ45_Abracon_ARJM11C7-114-BA-EW2 -> KM-Connector_RJ:Connector_RJ45_Abracon_ARJM11C7-114-BA-EW2
- L1: footprint (none) -> Inductor_SMD:L_1206_3216Metric
- Y1: footprint (none) -> Crystal:Crystal_SMD_HC49-SD_HandSoldering
Connections:
- net at U1.24 (OSC2): now also C14.2, Y1.1
Changed lines of the file:
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@@
-    (stroke (width 0) (type default))
-  )
-  (wire (pts (xy 125.73 84.455) (xy 128.27 84.455))
     (stroke (width 0) (type default))
   )
@@
     (stroke (width 0) (type default))
   )
-  (wire (pts (xy 133.35 84.455) (xy 161.29 84.455))
+  (wire (pts (xy 125.73 84.455) (xy 161.29 84.455))
     (stroke (width 0) (type default))
   )
@@
       (effects (font (size 1.27 1.27)) (justify right))
     )
-    (property "Footprint" "" (at 125.73 79.375 0)
+    (property "Footprint" "Crystal:Crystal_SMD_HC49-SD_HandSoldering" (at 125.73 79.375 0)
       (effects (font (size 1.27 1.27)) hide)
     )
@@
     )
   )
-  (symbol (lib_id "Device:R_Small") (at 130.81 84.455 90) (unit 1)
-    (in_bom yes) (on_board yes) (dnp no)
-    (property "Reference" "R16" (at 130.81 86.995 90)
-      (effects (font (size 1.27 1.27)))
-    )
-    (property "Value" "R_Small" (at 130.81 89.535 90)
-      (effects (font (size 1.27 1.27)))
-    )
-    (property "Footprint" "" (at 130.81 84.455 0)
-      (effects (font (size 1.27 1.27)) hide)
-    )
-    (property "Datasheet" "~" (at 130.81 84.455 0)
-      (effects (font (size 1.27 1.27)) hide)
-    )
-    (pin "1")
-    (pin "2")
-    (instances
-      (project "LED-driver-kicad"
-        (path "/2b071084-2ab6-4896-84cc-45b211479417"
-          (reference "R16") (unit 1)
-        )
-        (path "/2b071084-2ab6-4896-84cc-45b211479417/359e4c60-3d39-46c5-bd25-b25d83369b39"
-          (reference "R7") (unit 1)
-        )
-      )
-    )
-  )
   (symbol (lib_id "power:+3.3V") (at 158.75 42.545 0) (unit 1)
     (in_bom yes) (on_board yes) (dnp no)
@@
       (effects (font (size 1.27 1.27)))
     )
-    (property "Footprint" "Connector_RJ:Connector_RJ45_Abracon_ARJM11C7-114-BA-EW2" (at 51.435 79.375 0)
+    (property "Footprint" "KM-Connector_RJ:Connector_RJ45_Abracon_ARJM11C7-114-BA-EW2" (at 51.435 79.375 0)
       (effects (font (size 1.27 1.27) italic) hide)
     )
@@
       (effects (font (size 1.27 1.27)) (justify left))
     )
-    (property "Footprint" "" (at 247.015 77.47 0)
-      (effects (font (size 1.27 1.27)) hide)
-    )
+    (property "Footprint" "Inductor_SMD:L_1206_3216Metric" (at 247.015 77.47 0)
+      (effects (font (size 1.27 1.27)) hide)
+    )
