File: LED-driver-kicad/Ethernet.kicad_sch (KiCad schematic)
At the start: 22 parts, among them J1 ARJM11C7-114-BA-EW2, U1 ENC28J60x-SO, Y1 25MHz

Commit message: update initial components layout
Parts:
- Y1: footprint Crystal:Crystal_SMD_HC49-SD_HandSoldering -> Crystal:Crystal_SMD_HC49-SD
Changed lines of the file:
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@@
       (effects (font (size 1.27 1.27)) (justify right))
     )
-    (property "Footprint" "Crystal:Crystal_SMD_HC49-SD_HandSoldering" (at 125.73 79.375 0)
+    (property "Footprint" "Crystal:Crystal_SMD_HC49-SD" (at 125.73 79.375 0)
       (effects (font (size 1.27 1.27)) hide)
     )

Commit message: add test points, net ties to schematics
Parts:
- renumbered C6 to C2, C2 to C5, C3 to C6, C4 to C7
