File: LED-driver-kicad/LEDs.kicad_sch (KiCad schematic)
At the start: 54 parts, among them Q8 Q_NMOS_GDS, U6 MIC3205YML-TR, U7 MIC3205YML-TR, U8 MIC3205YML-TR

Commit message: update footprint assignments
Parts:
- D11, D12, D13, D14, D15, D16: footprint LED_SMD:LED_Cree-JE2835_3V_NClass -> KM-LED_SMD:LED_Cree-JE2835_3V_NClass_Group-2
- D18, D19, D20, D21, D22, D23, D25, D26, D27, D28, D29, D30: footprint LED_SMD:LED_Cree-JE2835_3V_NClass -> KM-LED_SMD:LED_Cree-JE2835_3V_NClass_Group-1
- Q8: footprint (none) -> KM-Package_SOT_SMD:SOT-23_Handsoldering
- U7, U8: footprint Mahabeer-Package_DFN_QFN:MLF-10_ML_MCH-Driver_LED_Microchip_MIC3205YML-TR -> KM-Package_DFN_QFN:MLF-10_ML_MCH-Driver_LED_Microchip_MIC3205YML-TR
Changed lines of the file:
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@@
       (effects (font (size 1.27 1.27)))
     )
-    (property "Footprint" "Mahabeer-Package_DFN_QFN:MLF-10_ML_MCH-Driver_LED_Microchip_MIC3205YML-TR" (at 205.105 115.57 0)
+    (property "Footprint" "KM-Package_DFN_QFN:MLF-10_ML_MCH-Driver_LED_Microchip_MIC3205YML-TR" (at 205.105 115.57 0)
       (effects (font (size 1.27 1.27) italic) hide)
     )
@@
       (effects (font (size 1.27 1.27)))
     )
-    (property "Footprint" "LED_SMD:LED_Cree-JE2835_3V_NClass" (at 211.455 73.025 90)
+    (property "Footprint" "KM-LED_SMD:LED_Cree-JE2835_3V_NClass_Group-1" (at 211.455 73.025 90)
       (effects (font (size 1.27 1.27)) hide)
     )
@@
       (effects (font (size 1.27 1.27)))
     )
-    (property "Footprint" "Mahabeer-Package_DFN_QFN:MLF-10_ML_MCH-Driver_LED_Microchip_MIC3205YML-TR" (at 78.105 166.37 0)
+    (property "Footprint" "KM-Package_DFN_QFN:MLF-10_ML_MCH-Driver_LED_Microchip_MIC3205YML-TR" (at 78.105 166.37 0)
       (effects (font (size 1.27 1.27) italic) hide)
     )
@@
       (effects (font (size 1.27 1.27)))
     )
-    (property "Footprint" "LED_SMD:LED_Cree-JE2835_3V_NClass" (at 218.44 73.025 90)
+    (property "Footprint" "KM-LED_SMD:LED_Cree-JE2835_3V_NClass_Group-1" (at 218.44 73.025 90)
       (effects (font (size 1.27 1.27)) hide)
     )
@@
       (effects (font (size 1.27 1.27)))
     )
-    (property "Footprint" "LED_SMD:LED_Cree-JE2835_3V_NClass" (at 70.485 123.825 90)
+    (property "Footprint" "KM-LED_SMD:LED_Cree-JE2835_3V_NClass_Group-1" (at 70.485 123.825 90)
       (effects (font (size 1.27 1.27)) hide)
     )
@@
       (effects (font (size 1.27 1.27)))
     )
-    (property "Footprint" "LED_SMD:LED_Cree-JE2835_3V_NClass" (at 86.36 41.275 90)
+    (property "Footprint" "KM-LED_SMD:LED_Cree-JE2835_3V_NClass_Group-2" (at 86.36 41.275 90)
       (effects (font (size 1.27 1.27)) hide)
     )
@@
       (effects (font (size 1.27 1.27)))
     )
-    (property "Footprint" "LED_SMD:LED_Cree-JE2835_3V_NClass" (at 76.2 41.275 90)
+    (property "Footprint" "KM-LED_SMD:LED_Cree-JE2835_3V_NClass_Group-2" (at 76.2 41.275 90)
       (effects (font (size 1.27 1.27)) hide)
     )
@@
       (effects (font (size 1.27 1.27)))
     )
-    (property "Footprint" "LED_SMD:LED_Cree-JE2835_3V_NClass" (at 224.79 73.025 90)
+    (property "Footprint" "KM-LED_SMD:LED_Cree-JE2835_3V_NClass_Group-1" (at 224.79 73.025 90)
       (effects (font (size 1.27 1.27)) hide)
     )
@@
       (effects (font (size 1.27 1.27)))
     )
-    (property "Footprint" "LED_SMD:LED_Cree-JE2835_3V_NClass" (at 66.04 41.275 90)
+    (property "Footprint" "KM-LED_SMD:LED_Cree-JE2835_3V_NClass_Group-2" (at 66.04 41.275 90)
       (effects (font (size 1.27 1.27)) hide)
     )
@@
       (effects (font (size 1.27 1.27)))
     )
-    (property "Footprint" "LED_SMD:LED_Cree-JE2835_3V_NClass" (at 84.455 123.825 90)
+    (property "Footprint" "KM-LED_SMD:LED_Cree-JE2835_3V_NClass_Group-1" (at 84.455 123.825 90)
       (effects (font (size 1.27 1.27)) hide)
     )
@@
       (effects (font (size 1.27 1.27)))
     )
-    (property "Footprint" "LED_SMD:LED_Cree-JE2835_3V_NClass" (at 91.44 41.275 90)
+    (property "Footprint" "KM-LED_SMD:LED_Cree-JE2835_3V_NClass_Group-2" (at 91.44 41.275 90)
       (effects (font (size 1.27 1.27)) hide)
     )
@@
       (effects (font (size 1.27 1.27)))
     )
-    (property "Footprint" "LED_SMD:LED_Cree-JE2835_3V_NClass" (at 91.44 123.825 90)
+    (property "Footprint" "KM-LED_SMD:LED_Cree-JE2835_3V_NClass_Group-1" (at 91.44 123.825 90)
       (effects (font (size 1.27 1.27)) hide)
     )
@@
       (effects (font (size 1.27 1.27)) (justify left))
     )
-    (property "Footprint" "" (at 120.015 142.24 0)
+    (property "Footprint" "KM-Package_SOT_SMD:SOT-23_Handsoldering" (at 120.015 142.24 0)
       (effects (font (size 1.27 1.27)) hide)
     )
@@
       (effects (font (size 1.27 1.27)))
     )
-    (property "Footprint" "LED_SMD:LED_Cree-JE2835_3V_NClass" (at 81.28 41.275 90)
+    (property "Footprint" "KM-LED_SMD:LED_Cree-JE2835_3V_NClass_Group-2" (at 81.28 41.275 90)
       (effects (font (size 1.27 1.27)) hide)
     )
@@
       (effects (font (size 1.27 1.27)))
     )
-    (property "Footprint" "LED_SMD:LED_Cree-JE2835_3V_NClass" (at 71.12 41.275 90)
+    (property "Footprint" "KM-LED_SMD:LED_Cree-JE2835_3V_NClass_Group-2" (at 71.12 41.275 90)
       (effects (font (size 1.27 1.27)) hide)
     )
@@
       (effects (font (size 1.27 1.27)))
     )
-    (property "Footprint" "LED_SMD:LED_Cree-JE2835_3V_NClass" (at 63.5 123.825 90)
+    (property "Footprint" "KM-LED_SMD:LED_Cree-JE2835_3V_NClass_Group-1" (at 63.5 123.825 90)
       (effects (font (size 1.27 1.27)) hide)
     )
@@
       (effects (font (size 1.27 1.27)))
     )
-    (property "Footprint" "LED_SMD:LED_Cree-JE2835_3V_NClass" (at 190.5 73.025 90)
+    (property "Footprint" "KM-LED_SMD:LED_Cree-JE2835_3V_NClass_Group-1" (at 190.5 73.025 90)
       (effects (font (size 1.27 1.27)) hide)
     )
@@
       (effects (font (size 1.27 1.27)))
     )
-    (property "Footprint" "LED_SMD:LED_Cree-JE2835_3V_NClass" (at 77.47 123.825 90)
+    (property "Footprint" "KM-LED_SMD:LED_Cree-JE2835_3V_NClass_Group-1" (at 77.47 123.825 90)
       (effects (font (size 1.27 1.27)) hide)
     )
@@
       (effects (font (size 1.27 1.27)))
     )
-    (property "Footprint" "LED_SMD:LED_Cree-JE2835_3V_NClass" (at 204.47 73.025 90)
+    (property "Footprint" "KM-LED_SMD:LED_Cree-JE2835_3V_NClass_Group-1" (at 204.47 73.025 90)
       (effects (font (size 1.27 1.27)) hide)
     )
@@
       (effects (font (size 1.27 1.27)))
     )
-    (property "Footprint" "LED_SMD:LED_Cree-JE2835_3V_NClass" (at 97.79 123.825 90)
+    (property "Footprint" "KM-LED_SMD:LED_Cree-JE2835_3V_NClass_Group-1" (at 97.79 123.825 90)
       (effects (font (size 1.27 1.27)) hide)
     )
@@
       (effects (font (size 1.27 1.27)))
     )
-    (property "Footprint" "LED_SMD:LED_Cree-JE2835_3V_NClass" (at 197.485 73.025 90)
+    (property "Footprint" "KM-LED_SMD:LED_Cree-JE2835_3V_NClass_Group-1" (at 197.485 73.025 90)
       (effects (font (size 1.27 1.27)) hide)
     )
@@
       (effects (font (size 1.27 1.27)) (justify left))
     )
-    (property "Footprint" "" (at 247.015 91.44 0)
+    (property "Footprint" "KM-Package_SOT_SMD:SOT-23_Handsoldering" (at 247.015 91.44 0)
       (effects (font (size 1.27 1.27)) hide)
     )
@@
       (effects (font (size 1.27 1.27)) (justify left))
     )
-    (property "Footprint" "" (at 120.015 59.69 0)
-      (effects (font (size 1.27 1.27)) hide)
-    )
+    (property "Footprint" "KM-Package_SOT_SMD:SOT-23_Handsoldering" (at 120.015 59.69 0)
+      (effects (font (size 1.27 1.27)) hide)
+    )
