File: LED-driver-kicad/LEDs-amber_white.kicad_sch (KiCad schematic)
At the start: 53 parts, among them Q4 Q_NMOS_GDS, Q5 Q_NMOS_GDS, Q6 Q_NMOS_GDS, U11 74AHC1G14, U7 MIC3205YML-TR

Commit message: initial PCB layout
Parts:
- D27: value BAT42 -> SD103AWS; footprint Diode_THT:D_DO-35_SOD27_P7.62mm_Horizontal -> Diode_SMD:D_SOD-323_HandSoldering; symbol Diode:BAT42 -> Device:D_Schottky_Small
Changed lines of the file:
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@@
-    (stroke (width 0) (type default))
-  )
-  (wire (pts (xy 83.185 31.75) (xy 121.92 31.75))
     (stroke (width 0) (type default))
   )
@@
     (stroke (width 0) (type default))
   )
-  (wire (pts (xy 47.625 127) (xy 75.565 127))
+  (wire (pts (xy 47.625 127) (xy 76.835 127))
     (stroke (width 0) (type default))
   )
@@
     (stroke (width 0) (type default))
   )
-  (wire (pts (xy 83.185 127) (xy 121.92 127))
+  (wire (pts (xy 81.915 127) (xy 121.92 127))
     (stroke (width 0) (type default))
   )
@@
     (stroke (width 0) (type default))
   )
-  (wire (pts (xy 47.625 31.75) (xy 75.565 31.75))
+  (wire (pts (xy 47.625 31.75) (xy 76.835 31.75))
     (stroke (width 0) (type default))
   )
@@
     (stroke (width 0) (type default))
   )
+  (wire (pts (xy 81.915 31.75) (xy 121.92 31.75))
+    (stroke (width 0) (type default))
+  )
   (wire (pts (xy 59.69 50.8) (xy 75.565 50.8))
     (stroke (width 0) (type default))
@@
     (stroke (width 0) (type default))
   )
-  (wire (pts (xy 174.625 31.75) (xy 202.565 31.75))
+  (wire (pts (xy 174.625 31.75) (xy 203.835 31.75))
     (stroke (width 0) (type default))
   )
@@
     (stroke (width 0) (type default))
   )
-  (wire (pts (xy 210.185 31.75) (xy 248.92 31.75))
+  (wire (pts (xy 208.915 31.75) (xy 248.92 31.75))
     (stroke (width 0) (type default))
   )
@@
     )
   )
-  (symbol (lib_id "Diode:BAT42") (at 206.375 31.75 0) (unit 1)
+  (symbol (lib_id "Device:D_Schottky_Small") (at 206.375 31.75 0) (unit 1)
     (in_bom yes) (on_board yes) (dnp no)
     (property "Reference" "D27" (at 206.375 26.67 0)
       (effects (font (size 1.27 1.27)))
     )
-    (property "Value" "BAT42" (at 206.375 29.21 0)
-      (effects (font (size 1.27 1.27)))
-    )
-    (property "Footprint" "Diode_THT:D_DO-35_SOD27_P7.62mm_Horizontal" (at 206.375 36.195 0)
-      (effects (font (size 1.27 1.27)) hide)
-    )
-    (property "Datasheet" "http://www.vishay.com/docs/85660/bat42.pdf" (at 206.375 31.75 0)
+    (property "Value" "SD103AWS" (at 206.375 29.21 0)
+      (effects (font (size 1.27 1.27)))
+    )
+    (property "Footprint" "Diode_SMD:D_SOD-323_HandSoldering" (at 206.375 31.75 90)
+      (effects (font (size 1.27 1.27)) hide)
+    )
+    (property "Datasheet" "~" (at 206.375 31.75 90)
       (effects (font (size 1.27 1.27)) hide)
     )
@@
     )
   )
-  (symbol (lib_id "Diode:BAT42") (at 79.375 127 0) (unit 1)
+  (symbol (lib_id "Device:D_Schottky_Small") (at 79.375 127 0) (unit 1)
     (in_bom yes) (on_board yes) (dnp no)
     (property "Reference" "D27" (at 79.375 121.92 0)
       (effects (font (size 1.27 1.27)))
     )
-    (property "Value" "BAT42" (at 79.375 124.46 0)
-      (effects (font (size 1.27 1.27)))
-    )
-    (property "Footprint" "Diode_THT:D_DO-35_SOD27_P7.62mm_Horizontal" (at 79.375 131.445 0)
-      (effects (font (size 1.27 1.27)) hide)
-    )
-    (property "Datasheet" "http://www.vishay.com/docs/85660/bat42.pdf" (at 79.375 127 0)
+    (property "Value" "SD103AWS" (at 79.375 124.46 0)
+      (effects (font (size 1.27 1.27)))
+    )
+    (property "Footprint" "Diode_SMD:D_SOD-323_HandSoldering" (at 79.375 127 90)
+      (effects (font (size 1.27 1.27)) hide)
+    )
+    (property "Datasheet" "~" (at 79.375 127 90)
       (effects (font (size 1.27 1.27)) hide)
     )
@@
     )
   )
-  (symbol (lib_id "Diode:BAT42") (at 79.375 31.75 0) (unit 1)
+  (symbol (lib_id "Device:D_Schottky_Small") (at 79.375 31.75 0) (unit 1)
     (in_bom yes) (on_board yes) (dnp no)
     (property "Reference" "D27" (at 79.375 26.67 0)
       (effects (font (size 1.27 1.27)))
     )
-    (property "Value" "BAT42" (at 79.375 29.21 0)
-      (effects (font (size 1.27 1.27)))
-    )
-    (property "Footprint" "Diode_THT:D_DO-35_SOD27_P7.62mm_Horizontal" (at 79.375 36.195 0)
-      (effects (font (size 1.27 1.27)) hide)
-    )
-    (property "Datasheet" "http://www.vishay.com/docs/85660/bat42.pdf" (at 79.375 31.75 0)
-      (effects (font (size 1.27 1.27)) hide)
-    )
+    (property "Value" "SD103AWS" (at 79.375 29.21 0)
+      (effects (font (size 1.27 1.27)))
+    )
+    (property "Footprint" "Diode_SMD:D_SOD-323_HandSoldering" (at 79.375 31.75 90)
+      (effects (font (size 1.27 1.27)) hide)
+    )
+    (property "Datasheet" "~" (at 79.375 31.75 90)
+      (effects (font (size 1.27 1.27)) hide)
+    )
