File: LED-driver-kicad/LED-driver-kicad.kicad_pcb (KiCad board)
At the start: 2 copper layers, 88.9 x 81.3 mm, 192 parts, among them J1 ARJM11C7-114-BA-EW2, J2 Conn_01x03_Socket, J3 Conn_01x03_Socket, J4 Conn_01x05_Socket, J5 Conn_01x02_Socket, Q1 Q_NMOS_GDS, Q2 Q_NMOS_GDS, Q3 Q_NMOS_GDS, Q4 Q_NMOS_GDS, Q5 Q_NMOS_GDS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

Commit message: update PCB version number
Other:
- board text added: "2537_5b7a_0023 LED DRIVER v1.0"
- board text removed: "2537_5b7a_0023 LED DRIVER v0.1"
Changed lines of the file:
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@@
     (effects (font (size 0.8 1) (thickness 0.153) bold) (justify left bottom))
   )
-  (gr_text "2537_5b7a_0023\nLED DRIVER\nv0.1" (at 94.234 52.578) (layer "F.SilkS" knockout)
+  (gr_text "2537_5b7a_0023\nLED DRIVER\nv1.0" (at 94.234 52.578) (layer "F.SilkS" knockout)
     (effects (font (size 1 1) (thickness 0.153) bold) (justify left bottom))
   )
